File: Hardware/ADC.brd (EAGLE design)
At the start: 50 x 50 mm, 61 parts, among them IC1 LTC2246, IC2 LP5907, IC3 74VCX16373, IC4 NC7SZ14P5X, IC5 NC7SZ14P5X, X1 SMA-142-0711-871/876, X2 SMA-142-0711-871/876

Commit message: Further experiments/scripts
Connections:
- net N$69 renamed SPI_NSS
- net N$70 renamed SPI_MOSI
- net N$71 renamed SPI_MISO
- net N$72 renamed SPI_SCK
Changed lines of the file:
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@@
 <wire x1="44.71" y1="19.9" x2="44.73" y2="19.92" width="0.3" layer="1"/>
 </signal>
-<signal name="N$69">
+<signal name="SPI_NSS">
 <contactref element="JP4" pad="5"/>
 <contactref element="JP4" pad="6"/>
@@
 <wire x1="43.46" y1="11.1" x2="46.07" y2="11.1" width="0.3" layer="16"/>
 </signal>
-<signal name="N$70">
+<signal name="SPI_MOSI">
 <contactref element="JP4" pad="8"/>
 <contactref element="JP4" pad="7"/>
@@
 <wire x1="42.12" y1="12.3" x2="44.73" y2="12.3" width="0.3" layer="16"/>
 </signal>
-<signal name="N$71">
+<signal name="SPI_MISO">
 <contactref element="JP4" pad="9"/>
 <contactref element="JP4" pad="10"/>
@@
 <wire x1="40.88" y1="13.6" x2="46.03" y2="13.6" width="0.3" layer="16"/>
 </signal>
-<signal name="N$72">
+<signal name="SPI_SCK">
 <contactref element="JP4" pad="12"/>
 <contactref element="JP4" pad="11"/>
