File: Hardware/ADC.sch (EAGLE design)
At the start: 61 parts, among them IC1 LTC2246, IC2 LP5907, IC3 74VCX16373, IC4 NC7SZ14P5X, IC5 NC7SZ14P5X, X1 SMA-142-0711-871/876, X2 SMA-142-0711-871/876

Commit message: Further experiments/scripts
Connections:
- net N$69 renamed SPI_NSS
- net N$70 renamed SPI_MOSI
- net N$71 renamed SPI_MISO
- net N$72 renamed SPI_SCK
Changed lines of the file:
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@@
 </segment>
 </net>
-<net name="N$69" class="0">
+<net name="SPI_NSS" class="0">
 <segment>
 <pinref part="JP4" gate="A" pin="5"/>
@@
 <pinref part="SV1" gate="1" pin="24"/>
 <wire x1="223.52" y1="50.8" x2="223.52" y2="43.18" width="0.1524" layer="91"/>
+<label x="236.22" y="50.8" size="1.778" layer="95"/>
 </segment>
 </net>
-<net name="N$70" class="0">
+<net name="SPI_MOSI" class="0">
 <segment>
 <pinref part="JP4" gate="A" pin="8"/>
@@
 <pinref part="SV1" gate="1" pin="23"/>
 <wire x1="223.52" y1="20.32" x2="223.52" y2="27.94" width="0.1524" layer="91"/>
+<label x="236.22" y="20.32" size="1.778" layer="95"/>
 </segment>
 </net>
-<net name="N$71" class="0">
+<net name="SPI_MISO" class="0">
 <segment>
 <pinref part="JP4" gate="A" pin="9"/>
@@
 <pinref part="SV1" gate="1" pin="22"/>
 <wire x1="220.98" y1="53.34" x2="220.98" y2="43.18" width="0.1524" layer="91"/>
+<label x="236.22" y="53.34" size="1.778" layer="95"/>
 </segment>
 </net>
-<net name="N$72" class="0">
+<net name="SPI_SCK" class="0">
 <segment>
 <pinref part="JP4" gate="A" pin="12"/>
@@
 <pinref part="SV1" gate="1" pin="21"/>
 <wire x1="220.98" y1="17.78" x2="220.98" y2="27.94" width="0.1524" layer="91"/>
+<label x="236.22" y="17.78" size="1.778" layer="95"/>
 </segment>
 </net>
