File: Hardware/Clockdistributor.brd (EAGLE design)
At the start: 50 x 50 mm, 40 parts, among them IC1 GRF4002, IC2 GRF4002, IC3 BGA2869, IC4 BGA2869, X1 IN, X2 OUT, X3 IN, X4 OUT, X5 IN, X6 OUT, X7 IN, X8 OUT

Commit message: More experimental PCB designs
Parts:
- removed C19: 10u, rcl:C1206
- removed IC1, IC2: GRF4002, rf:SON50P150X150X45-7T60X110
- removed IC3, IC4: BGA2869, rf:SOT363
- removed JP1: (no value), pinhead:1X02/90
- removed LED1: Green, eagle-ltspice:LED_SML0603
- added L7, L8: (no value), rcl:L2012C
- added R11, R12, R13, R14, R15, R16, R17, R18, R3, R4, R5, R6, R7, R8, R9: (no value), resistor:R0603
- C1, C3, C5, C7: value 100p -> (none)
- C10, C11, C12, C13, C14, C4, C8, C9: value 100n -> (none)
- C15, C16: value 10u -> (none); device rcl:C1206 -> rcl:C0603
- C2, C6: value 0p5 -> (none)
- L1, L2, L3, L4, L5, L6: value 100n -> (none); device resistor:R0603 -> rcl:L2012C
- R1, R2: value 6k5 -> (none)
- R10: value 220 -> (none)
- X1, X3, X5, X7: value IN -> SMA_CONNECTOR
- X2, X4, X6, X8: value OUT -> SMA_CONNECTOR
- moved R2 34.4 mm to (6.00, 40.0), turned to 0 degrees
- moved L6 33.1 mm to (42.5, 38.0), turned to 0 degrees
- moved C13 31.6 mm to (37.0, 45.0)
- moved C10 30.4 mm to (40.0, 13.0)
- moved L2 29.6 mm to (7.50, 12.0), turned to 180 degrees
- moved L5 28.6 mm to (42.5, 12.0), turned to 0 degrees
- moved L1 26.6 mm to (7.50, 38.0), turned to 180 degrees
- moved C12 25.7 mm to (40.0, 37.0)
- moved C14 25.1 mm to (37.0, 40.0), turned to 180 degrees
- moved C6 23.9 mm to (13.0, 10.0), turned to 0 degrees
- moved C2 23.9 mm to (10.0, 37.0), turned to 270 degrees
- moved X1 23.0 mm to (0.00, 38.0)
- moved X3 23.0 mm to (12.0, 0.00)
- moved X5 23.0 mm to (50.0, 12.0)
- moved X7 23.0 mm to (38.0, 50.0)
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Connections:
- removed net N$18: C13.2, X8.1
- removed net N$19: C4.1, L1.2, L3.1, R1.2
- removed net N$20: C8.1, L2.2, L4.1, R2.2
- removed net N$22: C14.1, IC4.1, L6.1
- removed net N$29: LED1.C, R10.2
- removed net VCC: C15.1, C16.1, C19.1, JP1.1, L3.2, L4.2, L5.2, L6.2, LED1.A
- net GND: now also C1.2, C10.2, C12.2, C13.2, C3.2, C5.2, C7.2, C9.2, R17.2, R18.2; no longer C19.2, IC1.2, IC1.5, IC1.6, IC1.7, IC2.2, IC2.5, IC2.6, IC2.7, IC3.2, IC3.4, IC3.5, IC4.2, IC4.4, IC4.5, JP1.2, R10.1
- net N$1: now also L1.2, R2.1
- net N$10: now also C10.1, L5.1, R9.1; no longer C7.2, X4.1
- net N$11: now also C11.1, L6.2, R12.1, X6.1; no longer C9.1, X5.1
- net N$12: now also C12.1, L6.1, R11.1; no longer C9.2, IC3.6
- net N$13: now also C13.1, L7.2, R14.1; no longer C12.1
- net N$14: now also C14.1, L7.1, R13.1; no longer C10.1, IC3.3
- net N$15: now also C15.1, L8.2, R16.1, X8.1; no longer C10.2, X6.1
- net N$16: now also C16.1, L8.1, R15.1; no longer C12.2, IC4.6
- net N$17: now also R10.2, R12.2, R14.2, R16.2, R17.1, R2.2, R4.2, R6.2, R8.2; no longer C13.1, IC4.3
- net N$2: now also C2.1, L1.1, R1.1; no longer C1.2, IC1.3
- net N$21: now also R1.2, R11.2, R13.2, R15.2, R18.1, R3.2, R5.2, R7.2, R9.2; no longer C11.1, IC3.1, L5.1
- net N$3: now also C3.1, L2.2, R4.1, X2.1; no longer IC1.1, R1.1
- net N$4: now also C4.1, L2.1, R3.1; no longer C2.1, C3.1, IC1.4, L1.1
- net N$5: now also C5.1, L3.2, R6.1, X3.1; no longer C3.2, X2.1
- net N$6: now also C6.1, L3.1, R5.1; no longer C5.1, X3.1
- net N$7: now also C7.1, L4.2, R8.1, X4.1; no longer C5.2, IC2.3
- net N$8: now also C8.1, L4.1, R7.1; no longer IC2.1, R2.1
- net N$9: now also C9.1, L5.2, R10.1, X5.1; no longer C6.1, C7.1, IC2.4, L2.1
Routing:
- net N$17: track 5.57 -> 120.6 mm, vias 0 -> 12
- net N$21: track 5.31 -> 84.4 mm
- net GND: track 28.9 -> 2.30 mm, vias 189 -> 43
- net VCC: track 21.5 -> 0.00 mm, vias 8 -> 0
- net N$20: track 6.30 -> 0.00 mm
- net N$19: track 6.30 -> 0.00 mm
- net N$22: track 5.41 -> 0.00 mm
- net N$18: track 4.03 -> 0.00 mm
- net N$4: track 9.25 -> 5.21 mm
- net N$9: track 9.19 -> 6.60 mm
- net N$15: track 4.03 -> 6.60 mm
- net N$13: track 4.03 -> 6.60 mm
- net N$11: track 4.03 -> 6.60 mm
- net N$1: track 4.05 -> 6.60 mm
- net N$5: track 4.08 -> 6.41 mm
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- removed copper zone on layer 2, net GND
- removed copper zone on layer 15, net VCC
Other:
- board text removed: "+15dB 0.1-3.8GHz"
- board text removed: "+31dB DC-2GHz"
- board text removed: "+5V"
- board text removed: "GND"
- board text removed: "Power"

Commit message: New Gerber files
Routing:
- net GND: track 2.30 -> 4.69 mm
Changed lines of the file:
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@@
 <grid distance="1" unitdist="mm" unit="mm" style="lines" multiple="1" display="yes" altdistance="5" altunitdist="mil" altunit="mil"/>
 <layers>
-<layer number="1" name="Top" color="4" fill="1" visible="no" active="yes"/>
+<layer number="1" name="Top" color="4" fill="1" visible="yes" active="yes"/>
 <layer number="2" name="Route2" color="16" fill="1" visible="no" active="no"/>
 <layer number="3" name="Route3" color="17" fill="1" visible="no" active="no"/>
@@
 <layer number="14" name="Route14" color="22" fill="1" visible="no" active="no"/>
 <layer number="15" name="Route15" color="23" fill="1" visible="no" active="no"/>
-<layer number="16" name="Bottom" color="1" fill="1" visible="no" active="yes"/>
+<layer number="16" name="Bottom" color="1" fill="1" visible="yes" active="yes"/>
 <layer number="17" name="Pads" color="2" fill="1" visible="yes" active="yes"/>
 <layer number="18" name="Vias" color="2" fill="1" visible="yes" active="yes"/>
-<layer number="19" name="Unrouted" color="6" fill="1" visible="no" active="yes"/>
+<layer number="19" name="Unrouted" color="6" fill="1" visible="yes" active="yes"/>
 <layer number="20" name="Dimension" color="24" fill="1" visible="yes" active="yes"/>
 <layer number="21" name="tPlace" color="7" fill="1" visible="yes" active="yes"/>
-<layer number="22" name="bPlace" color="7" fill="1" visible="no" active="yes"/>
-<layer number="23" name="tOrigins" color="15" fill="1" visible="no" active="yes"/>
-<layer number="24" name="bOrigins" color="15" fill="1" visible="no" active="yes"/>
-<layer number="25" name="tNames" color="7" fill="1" visible="yes" active="yes"/>
+<layer number="22" name="bPlace" color="7" fill="1" visible="yes" active="yes"/>
+<layer number="23" name="tOrigins" color="15" fill="1" visible="yes" active="yes"/>
+<layer number="24" name="bOrigins" color="15" fill="1" visible="yes" active="yes"/>
+<layer number="25" name="tNames" color="7" fill="1" visible="no" active="yes"/>
 <layer number="26" name="bNames" color="7" fill="1" visible="no" active="yes"/>
 <layer number="27" name="tValues" color="7" fill="1" visible="no" active="yes"/>
 <layer number="28" name="bValues" color="7" fill="1" visible="no" active="yes"/>
-<layer number="29" name="tStop" color="7" fill="3" visible="yes" active="yes"/>
+<layer number="29" name="tStop" color="7" fill="3" visible="no" active="yes"/>
 <layer number="30" name="bStop" color="7" fill="6" visible="no" active="yes"/>
 <layer number="31" name="tCream" color="7" fill="4" visible="no" active="yes"/>
@@
 <layer number="37" name="tTest" color="7" fill="1" visible="no" active="yes"/>
 <layer number="38" name="bTest" color="7" fill="1" visible="no" active="yes"/>
-<layer number="39" name="tKeepout" color="4" fill="11" visible="no" active="yes"/>
-<layer number="40" name="bKeepout" color="1" fill="11" visible="no" active="yes"/>
-<layer number="41" name="tRestrict" color="4" fill="10" visible="no" active="yes"/>
-<layer number="42" name="bRestrict" color="1" fill="10" visible="no" active="yes"/>
+<layer number="39" name="tKeepout" color="4" fill="11" visible="yes" active="yes"/>
+<layer number="40" name="bKeepout" color="1" fill="11" visible="yes" active="yes"/>
+<layer number="41" name="tRestrict" color="4" fill="10" visible="yes" active="yes"/>
+<layer number="42" name="bRestrict" color="1" fill="10" visible="yes" active="yes"/>
 <layer number="43" name="vRestrict" color="2" fill="10" visible="no" active="yes"/>
 <layer number="44" name="Drills" color="7" fill="1" visible="no" active="yes"/>
 <layer number="45" name="Holes" color="7" fill="1" visible="no" active="yes"/>
-<layer number="46" name="Milling" color="3" fill="1" visible="no" active="yes"/>
+<layer number="46" name="Milling" color="3" fill="1" visible="yes" active="yes"/>
 <layer number="47" name="Measures" color="7" fill="1" visible="no" active="yes"/>
 <layer number="48" name="Document" color="7" fill="1" visible="no" active="yes"/>
 <layer number="49" name="Reference" color="7" fill="1" visible="no" active="yes"/>
 <layer number="51" name="tDocu" color="7" fill="1" visible="yes" active="yes"/>
-<layer number="52" name="bDocu" color="7" fill="1" visible="no" active="yes"/>
+<layer number="52" name="bDocu" color="7" fill="1" visible="yes" active="yes"/>
 <layer number="88" name="SimResults" color="9" fill="1" visible="no" active="no"/>
 <layer number="89" name="SimProbes" color="9" fill="1" visible="no" active="no"/>
@@
 <wire x1="25" y1="25" x2="25" y2="26.15" width="1" layer="1"/>
 <via x="25" y="25" extent="1-16" drill="0.3" shape="octagon"/>
-<wire x1="8.5054" y1="2.1154" x2="8.5054" y2="2.1154" width="0" layer="19" extent="1-16"/>
 <via x="29" y="26" extent="1-16" drill="0.3" shape="octagon"/>
 <via x="31" y="28" extent="1-16" drill="0.3" shape="octagon"/>
@@
 <via x="26" y="25" extent="1-16" drill="0.3" shape="octagon"/>
 <via x="24" y="25" extent="1-16" drill="0.3" shape="octagon"/>
+<wire x1="8.5054" y1="2.1154" x2="8" y2="2.1154" width="0.3048" layer="1"/>
+<wire x1="8" y1="2.1154" x2="8" y2="4" width="0.3048" layer="1"/>
 </signal>
 <signal name="N$2">
@@
 <wire x1="10" y1="5.15" x2="11.95" y2="5.15" width="1" layer="1"/>
 <wire x1="11.95" y1="5.15" x2="12" y2="5.1" width="1" layer="1"/>
-<wire x1="12" y1="5.1" x2="12.15" y2="5" width="0" layer="19" extent="1-1"/>
+<wire x1="12.15" y1="5" x2="12" y2="5" width="0.3048" layer="1"/>
+<wire x1="12" y1="5" x2="12" y2="5.1" width="0.3048" layer="1"/>
 </signal>
 <signal name="N$6">
@@
 <contactref element="R7" pad="1"/>
 <contactref element="C8" pad="1"/>
-<wire x1="38" y1="8.5" x2="38" y2="11" width="1" layer="1"/>
+<wire x1="38" y1="8.5" x2="38" y2="10" width="1" layer="1"/>
+<wire x1="38" y1="10" x2="38" y2="11" width="1" layer="1"/>
 <wire x1="38" y1="11" x2="37" y2="12" width="1" layer="1"/>
 <wire x1="37" y1="12" x2="35.85" y2="12" width="1" layer="1"/>
-<wire x1="38" y1="11" x2="37.85" y2="10" width="0" layer="19" extent="1-1"/>
+<wire x1="37.85" y1="10" x2="38" y2="10" width="0.3048" layer="1"/>
 </signal>
 <signal name="N$9">
@@
 <mfgpreviewcolor name="substratecolor" color="0xFF786E46"/>
 </mfgpreviewcolors>
+<errors>
+</errors>
 </board>
 </drawing>
